Commit message: updated urdf files

File: lbr_da_vinci_endoscope/lbr_da_vinci_endoscope_description/urdf/lbr_da_vinci_endoscope.urdf.xacro (robot description, xacro)
@@ -3,20 +3,15 @@
 <robot xmlns:xacro="http://www.ros.org/wiki/xacro" name="lbr_da_vinci_endoscope">
     <!--Import the lbr med7 macro -->
-    <xacro:include filename="$(find lbr_description)/urdf/med7.xacro"/>
+    <xacro:include filename="$(find lbr_description)/urdf/med7/med7_description.urdf.xacro"/>
     <!-- Include endoscope xacro -->
-    <xacro:include filename="$(find da_vinci_endoscope_description)/urdf/da_vinci_endoscope.xacro"/>
+    <xacro:include filename="$(find da_vinci_endoscope_description)/urdf/da_vinci_endoscope_description.urdf.xacro"/>
     <!--  Arguments for the med7 macro  -->
-    <xacro:arg name="hardware_interface" default="PositionJointInterface"/>
     <xacro:arg name="robot_name" default="lbr"/>
-    <xacro:arg name="origin_xyz" default="0 0 0"/>
-    <xacro:arg name="origin_rpy" default="0 0 0"/>
     <!-- Arguments for endoscope xacro -->
     <xacro:arg name="endoscope_name" default="da_vinci_endoscope"/>
     <!-- fix to world -->
     <link name="world"/>
-    <!-- lbr -->
-    <xacro:med7 hardware_interface="$(arg hardware_interface)" parent="world" robot_name="$(arg robot_name)">
-        <origin xyz="$(arg origin_xyz)" rpy="$(arg origin_rpy)" />
-    </xacro:med7>
+    <!-- med -->
+    <xacro:med7 parent="world" robot_name="$(arg robot_name)" sim="$(arg sim)"/>
     <!-- insert endoscope -->
     <xacro:da_vinci_endoscope parent="$(arg robot_name)_link_ee" robot_name="$(arg robot_name)" endoscope_name="$(arg endoscope_name)"/>

File: lbr_storz_endoscope/lbr_storz_endoscope_description/urdf/lbr_storz_endoscope.urdf.xacro (robot description, xacro)
@@ -3,20 +3,15 @@
 <robot xmlns:xacro="http://www.ros.org/wiki/xacro" name="lbr_storz_endoscope">
     <!--Import the lbr med7 macro -->
-    <xacro:include filename="$(find lbr_description)/urdf/med7.xacro"/>
+    <xacro:include filename="$(find lbr_description)/urdf/med7/med7_description.urdf.xacro"/>
     <!-- Include endoscope xacro -->
-    <xacro:include filename="$(find storz_endoscope_description)/urdf/storz_endoscope.xacro"/>
+    <xacro:include filename="$(find storz_endoscope_description)/urdf/storz_endoscope_description.urdf.xacro"/>
     <!--  Arguments for the med7 macro  -->
-    <xacro:arg name="hardware_interface" default="PositionJointInterface"/>
     <xacro:arg name="robot_name" default="lbr"/>
-    <xacro:arg name="origin_xyz" default="0 0 0"/>
-    <xacro:arg name="origin_rpy" default="0 0 0"/>
     <!-- Arguments for endoscope xacro -->
     <xacro:arg name="endoscope_name" default="storz_endoscope"/>
     <!-- fix to world -->
     <link name="world"/>
-    <!-- lbr -->
-    <xacro:med7 hardware_interface="$(arg hardware_interface)" parent="world" robot_name="$(arg robot_name)">
-        <origin xyz="$(arg origin_xyz)" rpy="$(arg origin_rpy)" />
-    </xacro:med7>
+    <!-- med -->
+    <xacro:med7 parent="world" robot_name="$(arg robot_name)" sim="$(arg sim)"/>
     <!-- insert endoscope -->
     <xacro:storz_endoscope parent="$(arg robot_name)_link_ee" robot_name="$(arg robot_name)" endoscope_name="$(arg endoscope_name)"/>

File: lbr_storz_exoscope/lbr_storz_exoscope_description/urdf/lbr_storz_exoscope.urdf.xacro (robot description, xacro)
@@ -3,20 +3,15 @@
 <robot xmlns:xacro="http://www.ros.org/wiki/xacro" name="lbr_storz_exoscope">
     <!--Import the lbr med7 macro -->
-    <xacro:include filename="$(find lbr_description)/urdf/med7.xacro"/>
+    <xacro:include filename="$(find lbr_description)/urdf/med7/med7_description.urdf.xacro"/>
     <!-- Include exoscope xacro -->
-    <xacro:include filename="$(find storz_exoscope_description)/urdf/storz_exoscope.xacro"/>
+    <xacro:include filename="$(find storz_exoscope_description)/urdf/storz_exoscope_description.urdf.xacro"/>
     <!--  Arguments for the med7 macro  -->
-    <xacro:arg name="hardware_interface" default="PositionJointInterface"/>
     <xacro:arg name="robot_name" default="lbr"/>
-    <xacro:arg name="origin_xyz" default="0 0 0"/>
-    <xacro:arg name="origin_rpy" default="0 0 0"/>
     <!-- Arguments for exoscope xacro -->
     <xacro:arg name="exoscope_name" default="storz_exoscope"/>
     <!-- fix to world -->
     <link name="world"/>
-    <!-- lbr -->
-    <xacro:med7 hardware_interface="$(arg hardware_interface)" parent="world" robot_name="$(arg robot_name)">
-        <origin xyz="$(arg origin_xyz)" rpy="$(arg origin_rpy)" />
-    </xacro:med7>
+    <!-- med -->
+    <xacro:med7 parent="world" robot_name="$(arg robot_name)" sim="$(arg sim)"/>
     <!-- insert exoscope -->
     <xacro:storz_exoscope parent="$(arg robot_name)_link_ee" robot_name="$(arg robot_name)" exoscope_name="$(arg exoscope_name)"/>

File: lbr_storz_straight_exoscope_hsi/lbr_storz_straight_exoscope_hsi_description/urdf/lbr_storz_straight_exoscope_hsi.urdf.xacro (robot description, xacro)
@@ -3,20 +3,15 @@
 <robot xmlns:xacro="http://www.ros.org/wiki/xacro" name="lbr_storz_straight_exoscope_hsi">
     <!--Import the lbr med7 macro -->
-    <xacro:include filename="$(find lbr_description)/urdf/med7.xacro"/>
+    <xacro:include filename="$(find lbr_description)/urdf/med7/med7_description.urdf.xacro"/>
     <!-- Include exoscope xacro -->
-    <xacro:include filename="$(find storz_straight_exoscope_hsi_description)/urdf/storz_straight_exoscope_hsi.xacro"/>
+    <xacro:include filename="$(find storz_straight_exoscope_hsi_description)/urdf/storz_straight_exoscope_hsi_description.urdf.xacro"/>
     <!--  Arguments for the med7 macro  -->
-    <xacro:arg name="hardware_interface" default="PositionJointInterface"/>
     <xacro:arg name="robot_name" default="lbr"/>
-    <xacro:arg name="origin_xyz" default="0 0 0"/>
-    <xacro:arg name="origin_rpy" default="0 0 0"/>
     <!-- Arguments for exoscope xacro -->
     <xacro:arg name="exoscope_name" default="storz_straight_exoscope_hsi"/>
     <!-- fix to world -->
     <link name="world"/>
-    <!-- lbr -->
-    <xacro:med7 hardware_interface="$(arg hardware_interface)" parent="world" robot_name="$(arg robot_name)">
-        <origin xyz="$(arg origin_xyz)" rpy="$(arg origin_rpy)" />
-    </xacro:med7>
+    <!-- med -->
+    <xacro:med7 parent="world" robot_name="$(arg robot_name)" sim="$(arg sim)"/>
     <!-- insert exoscope -->
     <xacro:storz_straight_exoscope_hsi parent="$(arg robot_name)_link_ee" robot_name="$(arg robot_name)" exoscope_name="$(arg exoscope_name)"/>

File: lbr_storz_tilt_endoscope/lbr_storz_tilt_endoscope_description/urdf/lbr_storz_tilt_endoscope.urdf.xacro (robot description, xacro)
@@ -3,20 +3,15 @@
 <robot xmlns:xacro="http://www.ros.org/wiki/xacro" name="lbr_storz_tilt_endoscope">
     <!--Import the lbr med7 macro -->
-    <xacro:include filename="$(find lbr_description)/urdf/med7.xacro"/>
+    <xacro:include filename="$(find lbr_description)/urdf/med7/med7_description.urdf.xacro"/>
     <!-- Include tilt_endoscope xacro -->
-    <xacro:include filename="$(find storz_tilt_endoscope_description)/urdf/storz_tilt_endoscope.xacro"/>
+    <xacro:include filename="$(find storz_tilt_endoscope_description)/urdf/storz_tilt_endoscope_description.urdf.xacro"/>
     <!--  Arguments for the med7 macro  -->
-    <xacro:arg name="hardware_interface" default="PositionJointInterface"/>
     <xacro:arg name="robot_name" default="lbr"/>
-    <xacro:arg name="origin_xyz" default="0 0 0"/>
-    <xacro:arg name="origin_rpy" default="0 0 0"/>
     <!-- Arguments for tilt_endoscope xacro -->
     <xacro:arg name="tilt_endoscope_name" default="storz_tilt_endoscope"/>
     <!-- fix to world -->
     <link name="world"/>
-    <!-- lbr -->
-    <xacro:med7 hardware_interface="$(arg hardware_interface)" parent="world" robot_name="$(arg robot_name)">
-        <origin xyz="$(arg origin_xyz)" rpy="$(arg origin_rpy)" />
-    </xacro:med7>
+    <!-- med -->
+    <xacro:med7 parent="world" robot_name="$(arg robot_name)" sim="$(arg sim)"/>
     <!-- insert tilt_endoscope -->
     <xacro:storz_tilt_endoscope parent="$(arg robot_name)_link_ee" robot_name="$(arg robot_name)" tilt_endoscope_name="$(arg tilt_endoscope_name)"/>
